Commit message: update test model
simplfied graphics

File: models/test4/test.urdf (robot description, URDF)
Before this commit: robot excavator_urdf_ros2_ready, 9 links, 8 joints
Links:
- link excavator: geometry collision mesh filename=meshes/excavator_colliders_Mesh.obj scale=1. 1. 1.; visual mesh filename=meshes/excavator_colliders_Mesh.obj scale=1. 1. 1.
- link gripper_claw_1: geometry collision mesh filename=meshes/gripper_claw_1_colliders_Mesh.obj scale=1. 1. 1.; visual mesh filename=meshes/gripper_claw_1_colliders_Mesh.obj scale=1. 1. 1.
- link gripper_claw_2: geometry collision mesh filename=meshes/gripper_claw_2_colliders_Mesh.obj scale=1. 1. 1.; visual mesh filename=meshes/gripper_claw_2_colliders_Mesh.obj scale=1. 1. 1.
- link gripper_frame: geometry collision mesh filename=meshes/gripper_frame_colliders_Mesh.obj scale=1. 1. 1.; visual mesh filename=meshes/gripper_frame_colliders_Mesh.obj scale=1. 1. 1.
- link gripper_mount: geometry collision mesh filename=meshes/gripper_mount_colliders_Mesh.obj scale=1. 1. 1.; visual mesh filename=meshes/gripper_mount_colliders_Mesh.obj scale=1. 1. 1.
- link lift_boom: geometry collision mesh filename=meshes/lift_boom_colliders_Mesh.obj scale=1. 1. 1.; visual mesh filename=meshes/lift_boom_colliders_Mesh.obj scale=1. 1. 1.
- link tilt_boom: geometry collision mesh filename=meshes/tilt_boom_colliders_Mesh.obj scale=1. 1. 1.; visual mesh filename=meshes/tilt_boom_colliders_Mesh.obj scale=1. 1. 1.
- link tool_body: geometry collision mesh filename=meshes/tool_body_colliders_Mesh.obj scale=1. 1. 1.; visual mesh filename=meshes/tool_body_colliders_Mesh.obj scale=1. 1. 1.
- link upper_carriage: geometry collision mesh filename=meshes/upper_carriage_colliders_Mesh.obj scale=1. 1. 1.; visual mesh filename=meshes/upper_carriage_colliders_Mesh.obj scale=1. 1. 1.

Commit message: jonin testi

File: models/test4/test.urdf (robot description, URDF)
Before this commit: robot excavator_urdf_ros2_ready, 9 links, 8 joints
Joints:
- joint revolute_lift: origin xyz=0.0165 0. 0.0785 rpy=0. 0. 0. -> xyz=0.0165 0. 0.0785 rpy=0. -0.455181869 0.
- joint revolute_tilt: origin xyz=0.42008 0. -0.20564 rpy=0. 0. 0. -> xyz=0.42008 0. -0.20564 rpy=0. 0.455181869 0.
